File: ASCII16-X Mapper XL/ASCII16-X Mapper XL.kicad_pcb (KiCad board)
At the start: 2 copper layers, 99.8 x 65 mm, 40 parts, among them J1 MSX Cartridge Edge Fingers, U1 S29GL064S, U10 74LVC823A, U2 74LVC32A, U3 74LVC541A, U4 74LVC541A, U5 TLV1117LV33, U6 74LVC541A, U7 74HCT541, U8 74LVC139A, U9 74LVC823A

Commit message: Change LDO input / output caps to 10 µF.
The TLV1117LV33’s datasheet specifies input & output caps of 1 µF.
However the TLV1117LV33EVM-714 evaluation board has 10 µF caps, quote:

> The input and output capacitors for the TLV1117LVxx need be 0.4 μF (effective
> minimum) for stability; however, for conservative design practice accounting
> for widely varying noise environments, and dynamic line/load conditions, a
> 10-μF capacitor has been employed at the input and output ports.

See https://www.ti.com/lit/pdf/slvu449

Thanks to Wlcracks for the advice.
Parts:
- C5, C7: value 1 µF -> 10 µF
Changed lines of the file:
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@@
 			)
 		)
-		(property "Value" "1 µF"
+		(property "Value" "10 µF"
 			(at 8.05 0 90)
 			(layer "F.Fab")
@@
 			)
 		)
-		(property "Description" "CAP CER 1UF 25V X7R 10% 0805"
+		(property "Description" "CAP CER 10UF 16V X5R 10% 0805"
 			(at 0 0 270)
 			(unlocked yes)
@@
 			)
 		)
-		(property "MPN" "CL21B105KAFNNNE"
+		(property "MPN" "CL21A106KOQNNNE"
 			(at 0 0 0)
 			(layer "F.Fab")
@@
 			)
 		)
-		(property "Value" "1 µF"
+		(property "Value" "10 µF"
 			(at 8.05 0 90)
 			(layer "F.Fab")
@@
 			)
 		)
-		(property "Description" "CAP CER 1UF 25V X7R 10% 0805"
+		(property "Description" "CAP CER 10UF 16V X5R 10% 0805"
 			(at 0 0 270)
 			(unlocked yes)
@@
 			)
 		)
-		(property "MPN" "CL21B105KAFNNNE"
+		(property "MPN" "CL21A106KOQNNNE"
 			(at 0 0 0)
 			(layer "F.Fab")

Commit message: Increase noise tolerance on control signals.
Replacing the SN74LVC32A with a SN74LVC7032A with Schmitt inputs.

When the control lines are noisy, if the noise is so bad that it goes under the
threshold of 2 V logic high momentarily, this can produce false control signals.
Because the LVC series of logic gates have a fast propagation time they are much
more sensitive to this than LS or HCT series parts.

This has been observed with the MK 3.0 slot expander, whose 75 cm long ribbon
cable picks up a lot of noise, but it doesn’t buffer the signals. Under certain
conditions (unpowered, several other carts plugged in) the control signals can
dip under the threshold during Flash operations. This particularly affects the
/RESET, /RD and /WR lines; /SLTSL is locally generated and thus not affected.

The /RD and /WR signals are gated by /SLTSL so it is not an issue for them,
however a false transient /RESET signal will cause the mapper registers to
reset. The Flash chip is unaffected since reset must be held for 200 ns.

The SN74LVC7032A is a fairly new variant of the SN74LVC32A with Schmitt trigger
inputs. The hysteresis makes it more tolerant of noise. Tests have shown it
(almost) entirely eliminates the issue.
Parts:
- U2: value 74LVC32A -> 74LVC7032A
Changed lines of the file:
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@@
 			)
 		)
-		(property "Value" "74LVC32A"
+		(property "Value" "74LVC7032A"
 			(at 0 3.45 270)
 			(layer "F.Fab")
@@
 			)
 		)
-		(property "Datasheet" "http://www.ti.com/lit/gpn/SN74LVC32A"
+		(property "Datasheet" "http://www.ti.com/lit/gpn/SN74LVC7032A"
 			(at 0 0 90)
 			(unlocked yes)
@@
 			)
 		)
-		(property "Description" "IC GATE OR 4CH 2-INP 14TSSOP"
+		(property "Description" "IC GATE OR SCHMITT 4CH 2-INP 14TSSOP"
 			(at 0 0 90)
 			(unlocked yes)
@@
 			)
 		)
-		(property "MPN" "SN74LVC32APWR"
+		(property "MPN" "SN74LVC7032APWR"
 			(at 0 0 90)
 			(unlocked yes)
@@
 			)
 		)
-		(property "Substitutes" "Texas Instruments SN74LVC32APWT, Nexperia 74LVC32APW,118"
+		(property "Substitutes" "Texas Instruments SN74LVC32APWR, SN74LVC32APWT, Nexperia 74LVC32APW,118"
 			(at 0 0 90)
 			(unlocked yes)
